Commit message: change sample -> whill

File: whill_vehicle_description/urdf/vehicle.xacro (robot description, xacro)
@@ -2,5 +2,5 @@
 <robot xmlns:xacro="http://ros.org/wiki/xacro">
   <!-- load parameter -->
-  <xacro:property name="vehicle_info" value="${xacro.load_yaml('$(find sample_vehicle_description)/config/vehicle_info.param.yaml')}"/>
+  <xacro:property name="vehicle_info" value="${xacro.load_yaml('$(find whill_vehicle_description)/config/vehicle_info.param.yaml')}"/>
   <!-- vehicle body -->
   <link name="base_link">
@@ -8,5 +8,5 @@
       <origin xyz="${vehicle_info['/**']['ros__parameters']['wheel_base']/2.0} 0 0" rpy="${pi/2.0} 0 ${pi}"/>
       <geometry>
-        <mesh filename="package://sample_vehicle_description/mesh/lexus.dae" scale="1 1 1"/>
+        <mesh filename="package://whill_vehicle_description/mesh/lexus.dae" scale="1 1 1"/>
       </geometry>
     </visual>

Commit message: add wheel chair xacro

File: whill_vehicle_description/urdf/vehicle.xacro (robot description, xacro)
@@ -1,14 +1,235 @@
 <?xml version="1.0"?>
-<robot xmlns:xacro="http://ros.org/wiki/xacro">
-  <!-- load parameter -->
-  <xacro:property name="vehicle_info" value="${xacro.load_yaml('$(find whill_vehicle_description)/config/vehicle_info.param.yaml')}"/>
-  <!-- vehicle body -->
-  <link name="base_link">
-    <visual>
-      <origin xyz="${vehicle_info['/**']['ros__parameters']['wheel_base']/2.0} 0 0" rpy="${pi/2.0} 0 ${pi}"/>
-      <geometry>
-        <mesh filename="package://whill_vehicle_description/mesh/lexus.dae" scale="1 1 1"/>
-      </geometry>
-    </visual>
-  </link>
+<robot xmlns:xacro="http://www.ros.org/wiki/xacro" name="whill_modelc" >
+    <link name="base_link">
+        <inertial>
+          <mass value="83.7"/>
+          <origin xyz="0 0 0"/>
+          <inertia ixx="10.0" ixy="10.0" ixz="10.0" iyy="10.0" iyz="10.0" izz="100.0" />
+        </inertial>
+    </link>
+    <link name="base_floor">
+        <visual>
+            <geometry>
+                <box size="0.600 0.400 0.050"/>
+            </geometry>
+            <material name="grey">
+                <color rgba="0.5 0.5 0.5 1.0"/>
+            </material>
+        </visual>
+        <collision>
+            <geometry>
+                <box size="0.600 0.400 0.050"/>
+            </geometry>
+        </collision>
+        <inertial>
+            <origin xyz="0 0 0" rpy="0 0 0" />
+            <mass value="40" />
+            <inertia ixx="1.0"  ixy="0.0"   ixz="0.0"
+                                iyy="1.0"   iyz="0.0"
+                                            izz="1.0" />
+        </inertial>
+    </link>
+    <joint name="base_body_joint" type="fixed">
+        <parent link="base_link" />
+        <child link="base_floor" />
+        <origin xyz="0.3 0 0.0" rpy="0 0 0"/>
+    </joint>
+    <link name="footrest_link">
+        <collision>
+            <geometry>
+                <box size="0.250 0.260 0.050"/>
+            </geometry>
+        </collision>
+        <visual>
+            <geometry>
+                <box size="0.250 0.260 0.050"/>
+            </geometry>
+            <material name="grey">
+                <color rgba="0.5 0.5 0.5 1.0"/>
+            </material>
+        </visual>
+        <inertial>
+            <origin xyz="0 0 0" rpy="0 0 0" />
+            <mass value="1" />
+            <inertia ixx="1.0"  ixy="0.0"   ixz="0.0"
+                                iyy="1.0"   iyz="0.0"
+                                            izz="1.0" />
+        </inertial>
+    </link>
+    <joint name="footrest_joint" type="fixed">
+        <parent link="base_floor" />
+        <child link="footrest_link" />
+        <origin xyz="0.320 0 0" rpy="0 0 0"/>
+    </joint>
+    <link name="left_wheel_link">
+        <visual>
+            <geometry>
+                <cylinder length="0.05" radius="0.1325"/>
+            </geometry>
+            <origin xyz="0 0 0" rpy="0 0 0" />
+            <material name="black" />
+        </visual>
+        <collision>
+            <geometry>
+                <cylinder length="0.05" radius="0.1325"/>
+            </geometry>
+        </collision>
+        <inertial>
+            <origin xyz="0 0 0"/>
+            <mass value="0.500"/>
+            <inertia ixx="0.0013541667" ixy="0" ixz="0" iyy="0.0013541667" iyz="0" izz="0.0025"/>
+        </inertial>
+    </link>
+    <joint name="leftWheel" type="continuous">
+    <!--<joint name="leftWheel" type="fixed">-->
+        <parent link="base_floor" />
+        <child link="left_wheel_link" />
+        <origin xyz="-0.3 0.245 0" rpy="-1.57 0 0" />
+        <axis xyz="0 0 1" />
+    </joint>
+    <link name="right_wheel_link">
+        <collision>
+            <origin xyz="0 0 0" rpy="0 0 0" />
+            <geometry>
+                <cylinder length="0.05" radius="0.1325"/>
+            </geometry>
+        </collision>
+        <visual>
+            <origin xyz="0 0 0" rpy="0 0 0" />
+            <geometry>
+                <cylinder length="0.05" radius="0.1325"/>
+            </geometry>
+            <material name="black" />
+        </visual>
+        <inertial>
+            <origin xyz="0 0 0"/>
+            <mass value="0.500"/>
+            <inertia ixx="0.0013541667" ixy="0" ixz="0" iyy="0.0013541667" iyz="0" izz="0.0025"/>
+        </inertial>
+    </link>
+    <joint name="rightWheel" type="continuous">
+    <!--<joint name="rightWheel" type="fixed">-->
+        <parent link="base_floor" />
+        <child link="right_wheel_link" />
+        <origin xyz="-0.3 -0.245 0" rpy="1.57 0 0" />
+        <axis xyz="0 0 1" />
+    </joint>
+    <link name="frontwheel_left">
+        <collision>
+            <geometry>
+                <cylinder length="0.05" radius="0.1325"/>
+            </geometry>
+        </collision>
+        <visual>
+            <geometry>
+                <cylinder length="0.05" radius="0.1325"/>
+            </geometry>
+            <material name="black" />
+        </visual>
+        <inertial>
+            <origin xyz="0 0 0" rpy="0 0 0" />
+            <mass value="1.0" />
+            <inertia ixx="1.0"  ixy="0.0"   ixz="0.0"
+                                iyy="1.0"   iyz="0.0"
+                                            izz="1.0" />
+        </inertial>
+    </link>
+    <joint name="frontwheel_left_joint" type="fixed">
+        <parent link="base_floor" />
+        <child link="frontwheel_left" />
+        <origin xyz="0.3 -0.245 0" rpy="1.57 0 0" />
+        <axis xyz="0 0 1" />
+    </joint>
+    <link name="frontwheel_right">
+        <collision>
+            <geometry>
+                <cylinder length="0.05" radius="0.1325"/>
+            </geometry>
+        </collision>
+        <visual>
+            <geometry>
+                <cylinder length="0.05" radius="0.1325"/>
+            </geometry>
+            <material name="black" />
+        </visual>
+        <inertial>
+            <origin xyz="0 0 0" rpy="0 0 0" />
+            <mass value="1.0" />
+            <inertia ixx="1.0"  ixy="0.0"   ixz="0.0"
+                                iyy="1.0"   iyz="0.0"
+                                            izz="1.0" />
+        </inertial>
+    </link>
+    <joint name="frontwheel_right_joint" type="fixed">
+        <parent link="base_floor" />
+        <child link="frontwheel_right"/>
+        <origin xyz="0.3 0.245 0" rpy="1.57 0 0" />
+        <axis xyz="0 0 -1" />
+    </joint>
+    <!-- IMU -->
+    <link name="imu">
+    </link>
+    <joint name="imu_joint" type="fixed">
+        <axis xyz="0 1 0" />
+        <origin xyz="0.02 0 0.05" rpy="0 0.85521133347 3.14159265359"/>
+        <parent link="base_link"/>
+        <child link="imu"/>
+    </joint>
+    <!-- ===============  Transmission =============== -->
+    <transmission name="right_wheel_trans">
+        <type>transmission_interface/SimpleTransmission</type>
+        <joint name="rightWheel">
+            <hardwareInterface>hardware_interface/VelocityJointInterface</hardwareInterface>
+        </joint>
+        <actuator name="right_wheel_motor">
+            <hardwareInterface>hardware_interface/VelocityJointInterface</hardwareInterface>
+            <mechanicalReduction>30</mechanicalReduction>
+        </actuator>
+    </transmission>
+    <transmission name="left_wheel_trans">
+        <type>transmission_interface/SimpleTransmission</type>
+        <joint name="leftWheel">
+            <hardwareInterface>hardware_interface/VelocityJointInterface</hardwareInterface>
+        </joint>
+        <actuator name="left_wheel_motor">
+            <hardwareInterface>hardware_interface/VelocityJointInterface</hardwareInterface>
+            <mechanicalReduction>30</mechanicalReduction>
+        </actuator>
+    </transmission>
+    <!-- For Gazebo -->
+    <gazebo>
+        <plugin name="gazebo_ros_control" filename="libgazebo_ros_control.so">
+            <robotNamespace>/whill_simulator</robotNamespace>
+        </plugin>
+    </gazebo>
+    <gazebo reference="base_floor">
+        <selfCollide>true</selfCollide>
+        <mu1 value="0.05" />
+        <mu2 value="0.05" />
+    </gazebo>
+    <gazebo reference="sensor_arm_link">
+        <selfCollide>true</selfCollide>
+        <mu1 value="0.05" />
+        <mu2 value="0.05" />
+    </gazebo>
+    <gazebo reference="rearwheel_right">
+        <selfCollide>true</selfCollide>
+        <mu1 value="1.0" />
+        <mu2 value="1.0" />
+    </gazebo>
+    <gazebo reference="rearwheel_left">
+        <selfCollide>true</selfCollide>
+        <mu1 value="1.0" />
+        <mu2 value="1.0" />
+    </gazebo>
+    <gazebo reference="frontwheel_right">
+        <selfCollide>true</selfCollide>
+        <mu1 value="0.0" />
+        <mu2 value="0.0" />
+    </gazebo>
+    <gazebo reference="frontwheel_left">
+        <selfCollide>true</selfCollide>
+        <mu1 value="0.0" />
+        <mu2 value="0.0" />
+    </gazebo>
 </robot>

Commit message: fixed

File: whill_vehicle_description/urdf/vehicle.xacro (robot description, xacro)
@@ -81,6 +81,6 @@
         </inertial>
     </link>
-    <joint name="leftWheel" type="continuous">
-    <!--<joint name="leftWheel" type="fixed">-->
+    <!-- <joint name="leftWheel" type="continuous"> -->
+    <joint name="leftWheel" type="fixed">
         <parent link="base_floor" />
         <child link="left_wheel_link" />
@@ -108,6 +108,6 @@
         </inertial>
     </link>
-    <joint name="rightWheel" type="continuous">
-    <!--<joint name="rightWheel" type="fixed">-->
+    <!-- <joint name="rightWheel" type="continuous"> -->
+    <joint name="rightWheel" type="fixed">
         <parent link="base_floor" />
         <child link="right_wheel_link" />

Commit message: temporary solution:change parameter

File: whill_vehicle_description/urdf/vehicle.xacro (robot description, xacro)
@@ -81,6 +81,5 @@
         </inertial>
     </link>
-    <!-- <joint name="leftWheel" type="continuous"> -->
-    <joint name="leftWheel" type="fixed">
+    <joint name="leftWheel" type="continuous">
         <parent link="base_floor" />
         <child link="left_wheel_link" />
@@ -108,6 +107,5 @@
         </inertial>
     </link>
-    <!-- <joint name="rightWheel" type="continuous"> -->
-    <joint name="rightWheel" type="fixed">
+    <joint name="rightWheel" type="continuous">
         <parent link="base_floor" />
         <child link="right_wheel_link" />
